Commit message: Merda dos erros causados pelo gripper do moveit CORRIGIDOS.

File: panda_gz_moveit2/panda_description/urdf/panda.urdf (robot description, URDF)
Before this commit: robot panda, 14 links, 13 joints
Joints:
- joint panda_finger_joint1: limit lower=0 upper=0.04 effort=20 velocity=0.2 -> lower=-0.01 upper=0.042 effort=20 velocity=0.2
- joint panda_finger_joint2: limit lower=0 upper=0.04 effort=20 velocity=0.2 -> lower=-0.01 upper=0.042 effort=20 velocity=0.2

File: panda_gz_moveit2/panda_description/urdf/panda_gripper.xacro (robot description, xacro)
@@ -19,6 +19,6 @@
   <xacro:property name="joint_finger1_origin_rpy" value="0 0 0"/>
   <xacro:property name="joint_finger1_axis_xyz" value="0 1 0"/>
-  <xacro:property name="joint_finger1_lower_limit" value="0"/>
-  <xacro:property name="joint_finger1_upper_limit" value="0.04"/>
+  <xacro:property name="joint_finger1_lower_limit" value="-0.01"/>
+  <xacro:property name="joint_finger1_upper_limit" value="0.042"/>
   <xacro:property name="joint_finger1_velocity_limit" value="0.2"/>
   <xacro:property name="joint_finger1_torque_limit" value="20"/>
@@ -33,6 +33,6 @@
   <xacro:property name="joint_finger2_origin_rpy" value="0 0 0"/>
   <xacro:property name="joint_finger2_axis_xyz" value="0 -1 0"/>
-  <xacro:property name="joint_finger2_lower_limit" value="0"/>
-  <xacro:property name="joint_finger2_upper_limit" value="0.04"/>
+  <xacro:property name="joint_finger2_lower_limit" value="-0.01"/>
+  <xacro:property name="joint_finger2_upper_limit" value="0.042"/>
   <xacro:property name="joint_finger2_velocity_limit" value="0.2"/>
   <xacro:property name="joint_finger2_torque_limit" value="20"/>

File: panda_gz_moveit2/panda_moveit_config/srdf/panda_gripper.xacro (robot description, xacro)
@@ -16,10 +16,10 @@
     </group>
     <group_state name="open" group="gripper">
-      <joint name="${prefix}finger_joint1" value="0.04"/>
-      <joint name="${prefix}finger_joint2" value="0.04"/>
+      <joint name="${prefix}finger_joint1" value="0.042"/>
+      <joint name="${prefix}finger_joint2" value="0.042"/>
     </group_state>
     <group_state name="close" group="gripper">
-      <joint name="${prefix}finger_joint1" value="0.0"/>
-      <joint name="${prefix}finger_joint2" value="0.0"/>
+      <joint name="${prefix}finger_joint1" value="-0.01"/>
+      <joint name="${prefix}finger_joint2" value="-0.01"/>
     </group_state>
     <disable_collisions link1="${prefix}hand" link2="${prefix}leftfinger" reason="Adjacent"/>

Commit message: Atualização de colisão adicionada.

File: panda_gz_moveit2/panda_description/urdf/panda.urdf (robot description, URDF)
Before this commit: robot panda, 14 links, 13 joints
Joints:
- joint panda_joint2: limit lower=-1.7627825445142729 upper=1.7627825445142729 effort=87 velocity=2.6179938779914944 -> lower=-1.61277 upper=1.61277 effort=87 velocity=2.6179938779914944
