Commit message: Toma aí.

File: panda_gz_moveit2/panda_description/urdf/panda_arm.xacro (robot description, xacro)
@@ -19,6 +19,6 @@
   <xacro:property name="joint1_origin_rpy" value="0 0 0"/>
   <xacro:property name="joint1_axis_xyz" value="0 0 1"/>
-  <xacro:property name="joint1_lower_limit" value="${-166*pi/180}"/>
-  <xacro:property name="joint1_upper_limit" value="${166*pi/180}"/>
+  <xacro:property name="joint1_lower_limit" value="${-186*pi/180}"/>
+  <xacro:property name="joint1_upper_limit" value="${186*pi/180}"/>
   <xacro:property name="joint1_velocity_limit" value="${150*pi/180}"/>
   <xacro:property name="joint1_torque_limit" value="87"/>
@@ -32,6 +32,6 @@
   <xacro:property name="joint2_origin_rpy" value="${-pi/2} 0 0"/>
   <xacro:property name="joint2_axis_xyz" value="0 0 1"/>
-  <xacro:property name="joint2_lower_limit" value="${-101*pi/180}"/>
-  <xacro:property name="joint2_upper_limit" value="${101*pi/180}"/>
+  <xacro:property name="joint2_lower_limit" value="${-111*pi/180}"/>
+  <xacro:property name="joint2_upper_limit" value="${111*pi/180}"/>
   <xacro:property name="joint2_velocity_limit" value="${150*pi/180}"/>
   <xacro:property name="joint2_torque_limit" value="87"/>
@@ -45,6 +45,6 @@
   <xacro:property name="joint3_origin_rpy" value="${pi/2} 0 0"/>
   <xacro:property name="joint3_axis_xyz" value="0 0 1"/>
-  <xacro:property name="joint3_lower_limit" value="${-166*pi/180}"/>
-  <xacro:property name="joint3_upper_limit" value="${166*pi/180}"/>
+  <xacro:property name="joint3_lower_limit" value="${-186*pi/180}"/>
+  <xacro:property name="joint3_upper_limit" value="${186*pi/180}"/>
   <xacro:property name="joint3_velocity_limit" value="${150*pi/180}"/>
   <xacro:property name="joint3_torque_limit" value="87"/>
@@ -58,6 +58,6 @@
   <xacro:property name="joint4_origin_rpy" value="${pi/2} 0 0"/>
   <xacro:property name="joint4_axis_xyz" value="0 0 1"/>
-  <xacro:property name="joint4_lower_limit" value="${-176/180*pi}"/>
-  <xacro:property name="joint4_upper_limit" value="${-4/180*pi}"/>
+  <xacro:property name="joint4_lower_limit" value="${-186/180*pi}"/>
+  <xacro:property name="joint4_upper_limit" value="${-10/180*pi}"/>
   <xacro:property name="joint4_velocity_limit" value="${150*pi/180}"/>
   <xacro:property name="joint4_torque_limit" value="87"/>
@@ -71,6 +71,6 @@
   <xacro:property name="joint5_origin_rpy" value="${-pi/2} 0 0"/>
   <xacro:property name="joint5_axis_xyz" value="0 0 1"/>
-  <xacro:property name="joint5_lower_limit" value="${-166*pi/180}"/>
-  <xacro:property name="joint5_upper_limit" value="${166*pi/180}"/>
+  <xacro:property name="joint5_lower_limit" value="${-186*pi/180}"/>
+  <xacro:property name="joint5_upper_limit" value="${186*pi/180}"/>
   <xacro:property name="joint5_velocity_limit" value="${pi}"/>
   <xacro:property name="joint5_torque_limit" value="12"/>
@@ -84,6 +84,6 @@
   <xacro:property name="joint6_origin_rpy" value="${pi/2} 0 0"/>
   <xacro:property name="joint6_axis_xyz" value="0 0 1"/>
-  <xacro:property name="joint6_lower_limit" value="${-1/180*pi}"/>
-  <xacro:property name="joint6_upper_limit" value="${215/180*pi}"/>
+  <xacro:property name="joint6_lower_limit" value="${-4/180*pi}"/>
+  <xacro:property name="joint6_upper_limit" value="${315/180*pi}"/>
   <xacro:property name="joint6_velocity_limit" value="${pi}"/>
   <xacro:property name="joint6_torque_limit" value="12"/>
@@ -97,6 +97,6 @@
   <xacro:property name="joint7_origin_rpy" value="${pi/2} 0 0"/>
   <xacro:property name="joint7_axis_xyz" value="0 0 1"/>
-  <xacro:property name="joint7_lower_limit" value="${-166*pi/180}"/>
-  <xacro:property name="joint7_upper_limit" value="${166*pi/180}"/>
+  <xacro:property name="joint7_lower_limit" value="${-186*pi/180}"/>
+  <xacro:property name="joint7_upper_limit" value="${186*pi/180}"/>
   <xacro:property name="joint7_velocity_limit" value="${pi}"/>
   <xacro:property name="joint7_torque_limit" value="12"/>
