Commit message: Algoritmo simples para pegar e largar implementado.

File: moveit_resources/panda_description/urdf/panda.urdf (robot description, URDF)
Before this commit: robot panda, 12 links, 11 joints
Joints:
- joint panda_finger_joint1: limit lower=-0.02 upper=0.04 effort=20 velocity=0.2 -> lower=-0.02 upper=0.04 effort=200 velocity=0.2
- joint panda_finger_joint2: limit lower=-0.02 upper=0.04 effort=20 velocity=0.2 -> lower=-0.02 upper=0.04 effort=200 velocity=0.2; mimic joint=panda_finger_joint1 -> (none)

File: moveit_resources/panda_description/urdf/panda.urdf.xacro (robot description, xacro)
@@ -274,5 +274,5 @@
         <origin rpy="0 0 0" xyz="0 0 0.0584" />
         <axis xyz="0 1 0" />
-        <limit effort="20" lower="-0.02" upper="0.04" velocity="0.2" />
+        <limit effort="200" lower="-0.02" upper="0.04" velocity="0.2" />
         <dynamics damping="0.3" />
     </joint>
@@ -282,6 +282,5 @@
         <origin rpy="0 0 0" xyz="0 0 0.0584" />
         <axis xyz="0 -1 0" />
-        <limit effort="20" lower="-0.02" upper="0.04" velocity="0.2" />
-        <mimic joint="panda_finger_joint1" />
+        <limit effort="200" lower="-0.02" upper="0.04" velocity="0.2" />
         <dynamics damping="0.3" />
     </joint>

File: moveit_resources/panda_moveit_config/config/panda.ros2_control.xacro (robot description, xacro)
@@ -86,4 +86,13 @@
                 </state_interface>
             </joint>
+            <joint name="panda_finger_joint2">
+                <command_interface name="position" />
+                <state_interface name="position">
+                  <param name="initial_value">0.005</param>
+                </state_interface>
+                <state_interface name="velocity">
+                    <param name="initial_value">0.0</param>
+                </state_interface>
+            </joint>
         </ros2_control>
     </xacro:macro>

Commit message: Robustez do algoritmo de pegar e largar aumentada por meio do loop de retentativa do planejamento de trajetória do moveit.

File: moveit_resources/panda_description/urdf/panda.urdf (robot description, URDF)
Before this commit: robot panda, 12 links, 11 joints
Joints:
- joint panda_finger_joint1: limit lower=-0.02 upper=0.04 effort=200 velocity=0.2 -> lower=-0.02 upper=0.04 effort=50 velocity=0.2
- joint panda_finger_joint2: limit lower=-0.02 upper=0.04 effort=200 velocity=0.2 -> lower=-0.02 upper=0.04 effort=50 velocity=0.2

File: moveit_resources/panda_description/urdf/panda.urdf.xacro (robot description, xacro)
@@ -274,5 +274,5 @@
         <origin rpy="0 0 0" xyz="0 0 0.0584" />
         <axis xyz="0 1 0" />
-        <limit effort="200" lower="-0.02" upper="0.04" velocity="0.2" />
+        <limit effort="50" lower="-0.02" upper="0.04" velocity="0.2" />
         <dynamics damping="0.3" />
     </joint>
@@ -282,5 +282,5 @@
         <origin rpy="0 0 0" xyz="0 0 0.0584" />
         <axis xyz="0 -1 0" />
-        <limit effort="200" lower="-0.02" upper="0.04" velocity="0.2" />
+        <limit effort="50" lower="-0.02" upper="0.04" velocity="0.2" />
         <dynamics damping="0.3" />
     </joint>
