Commit message: Configuração de TF e ajustes em algumas configurações do Moveit para múltiplos robôs.

File: moveit_resources/panda_moveit_config/xacro_config/multi_robots.srdf.xacro (robot description, xacro)
@@ -2,6 +2,8 @@
 <robot xmlns:xacro="http://wiki.ros.org/xacro" name="multi_panda_system">
   <xacro:include filename="panda.srdf.xacro" />
-  <xacro:panda_srdf prefix="robot1_" />
-  <xacro:panda_srdf prefix="robot2_" />
-  <xacro:panda_srdf prefix="robot3_" />
+  <!-- Robot1: base móvel - usa virtual joint "planar" -->
+  <xacro:panda_srdf prefix="robot1_" virtual_joint_type="floating" />
+  <!-- Robot2 e Robot3: fixos - usa virtual joint "fixed" -->
+  <xacro:panda_srdf prefix="robot2_" virtual_joint_type="fixed" />
+  <xacro:panda_srdf prefix="robot3_" virtual_joint_type="fixed" />
 </robot>

File: moveit_resources/panda_moveit_config/xacro_config/multi_robots.urdf.xacro (robot description, xacro)
@@ -10,6 +10,7 @@
         initial_positions_file="$(arg initial_positions_file)"
         ros2_control_hardware_type="$(arg ros2_control_hardware_type)">
-        <origin xyz="0 0 0.01" rpy="0 0 0" />
+        <origin xyz="0 0 0.0" rpy="0 0 0" />
     </xacro:panda_system_multi>
+    <!-- ROBOT2 e ROBOT3: Fixos no world -->
     <xacro:panda_system_multi
         prefix="robot2_"

File: moveit_resources/panda_moveit_config/xacro_config/panda.srdf.xacro (robot description, xacro)
@@ -1,5 +1,5 @@
 <?xml version="1.0" encoding="UTF-8"?>
 <robot xmlns:xacro="http://wiki.ros.org/xacro">
-  <xacro:macro name="panda_srdf" params="prefix">
+  <xacro:macro name="panda_srdf" params="prefix virtual_joint_type:='fixed'">
     <group name="${prefix}panda_arm">
       <chain base_link="${prefix}panda_link0" tip_link="${prefix}panda_link8" />
@@ -53,5 +53,6 @@
         <joint name="${prefix}panda_finger_joint2" value="0.0"/>
     </group_state>
-    <virtual_joint name="${prefix}virtual_joint" type="fixed" parent_frame="world" child_link="${prefix}panda_link0" />
+    <!-- Virtual joint com tipo parametrizável -->
+    <virtual_joint name="${prefix}virtual_joint" type="floating" parent_frame="world" child_link="${prefix}panda_link0" />
     <disable_collisions link1="${prefix}panda_link0" link2="${prefix}panda_link1" reason="Adjacent"/>
     <disable_collisions link1="${prefix}panda_link0" link2="${prefix}panda_link2" reason="Never"/>

File: moveit_resources/panda_moveit_config/xacro_config/panda_system_macro.urdf.xacro (robot description, xacro)
@@ -4,5 +4,5 @@
   <xacro:include filename="panda.ros2_control.xacro" />
   <xacro:macro name="panda_system_multi" params="prefix parent *origin initial_positions_file ros2_control_hardware_type">
-    <joint name="${prefix}base_joint" type="fixed">
+    <joint name="${prefix}base_joint" type="floating">
       <xacro:insert_block name="origin" />
       <parent link="${parent}" />
